Commit message: update xacro names

File: imcoders_description/urdf/diff_wheeled_robot_with_IMcoders.xacro (robot description, xacro)
@@ -169,5 +169,5 @@
   <wheel fb="front" lr="left" parent="base_link" translateX="0" translateY="-0.5" flipY="1"/>
   <!-- IMcoder left -->
-  <link name="imu_left_link">
+  <link name="imcoder_left_link">
     <visual>
       <origin xyz="0 0 0" rpy="${M_PI/2} 0 0" />
@@ -178,12 +178,12 @@
     </visual>
   </link>
-  <joint name="imu_left_joint" type="fixed">
+  <joint name="imcoder_left_joint" type="fixed">
     <origin xyz="0 -${wheel_height/2 + imcoder_height/2} 0" rpy="0 0 0" />
     <parent link="front_left_wheel"/>
-    <child link="imu_left_link" />
+    <child link="imcoder_left_link" />
   </joint>
-  <gazebo reference="imu_left_link">
+  <gazebo reference="imcoder_left_link">
     <gravity>true</gravity>
-    <sensor name="imu_left_sensor" type="imu">
+    <sensor name="imcoder_left_sensor" type="imu">
       <always_on>true</always_on>
       <update_rate>100</update_rate>
@@ -191,11 +191,11 @@
       <topic>__default_topic__</topic>
       <plugin filename="libgazebo_ros_imu_sensor.so" name="imu_plugin">
-        <topicName>imu_left</topicName>
-        <bodyName>imu_left_link</bodyName>
+        <topicName>imcoder_left</topicName>
+        <bodyName>imcoder_left_link</bodyName>
         <updateRateHZ>10.0</updateRateHZ>
         <gaussianNoise>0.0</gaussianNoise>
         <xyzOffset>0 0 0</xyzOffset>
         <rpyOffset>0 0 0</rpyOffset>
-        <frameName>imu_left_link</frameName>
+        <frameName>imcoder_left_link</frameName>
       </plugin>
       <pose>0 0 0 0 0 0</pose>
@@ -203,5 +203,5 @@
   </gazebo>
   <!-- IMcoder right -->
-  <link name="imu_right_link">
+  <link name="imcoder_right_link">
     <visual>
       <origin xyz="0 0 0" rpy="${M_PI/2} 0 0" />
@@ -212,12 +212,12 @@
     </visual>
   </link>
-  <joint name="imu_right_joint" type="fixed">
+  <joint name="imcoder_right_joint" type="fixed">
     <origin xyz="0 ${wheel_height/2 + imcoder_height/2} 0" rpy="0 0 0" />
     <parent link="front_right_wheel"/>
-    <child link="imu_right_link" />
+    <child link="imcoder_right_link" />
   </joint>
-  <gazebo reference="imu_right_link">
+  <gazebo reference="imcoder_right_link">
     <gravity>true</gravity>
-    <sensor name="imu_right_sensor" type="imu">
+    <sensor name="imcoder_right_sensor" type="imu">
       <always_on>true</always_on>
       <update_rate>100</update_rate>
@@ -225,11 +225,11 @@
       <topic>__default_topic__</topic>
       <plugin filename="libgazebo_ros_imu_sensor.so" name="imu_plugin">
-        <topicName>imu_right</topicName>
-        <bodyName>imu_right_link</bodyName>
+        <topicName>imcoder_right</topicName>
+        <bodyName>imcoder_right_link</bodyName>
         <updateRateHZ>10.0</updateRateHZ>
         <gaussianNoise>0.0</gaussianNoise>
         <xyzOffset>0 0 0</xyzOffset>
         <rpyOffset>0 0 0</rpyOffset>
-        <frameName>imu_right_link</frameName>
+        <frameName>imcoder_right_link</frameName>
       </plugin>
       <pose>0 0 0 0 0 0</pose>

Commit message: Vector3 patch for odometry

File: imcoders_description/urdf/diff_wheeled_robot_with_IMcoders.xacro (robot description, xacro)
@@ -45,4 +45,8 @@
   <xacro:property name="imcoder_height" value="0.00545" />
   <xacro:property name="imcoder_radius" value="0.02" />
+  <!-- Update rates from plugin sensor. -->
+  <!-- Note that must be always [sensor_update_rate >= plugin_update_rate] -->
+  <xacro:property name="sensor_update_rate" value="100.0"/>
+  <xacro:property name="plugin_update_rate" value="100.0"/>
   <!-- Macro for calculating inertia of cylinder -->
   <xacro:macro name="cylinder_inertia" params="m r h">
@@ -187,5 +191,5 @@
     <sensor name="imu_left_sensor" type="imu">
       <always_on>true</always_on>
-      <update_rate>100</update_rate>
+      <update_rate>${sensor_update_rate}</update_rate>
       <visualize>true</visualize>
       <topic>__default_topic__</topic>
@@ -193,5 +197,5 @@
         <topicName>imu_left</topicName>
         <bodyName>imu_left_link</bodyName>
-        <updateRateHZ>100.0</updateRateHZ>
+        <updateRateHZ>${plugin_update_rate}</updateRateHZ>
         <gaussianNoise>0.0</gaussianNoise>
         <xyzOffset>0 0 0</xyzOffset>
@@ -221,5 +225,5 @@
     <sensor name="imu_right_sensor" type="imu">
       <always_on>true</always_on>
-      <update_rate>100</update_rate>
+      <update_rate>${sensor_update_rate}</update_rate>
       <visualize>true</visualize>
       <topic>__default_topic__</topic>
@@ -227,5 +231,5 @@
         <topicName>imu_right</topicName>
         <bodyName>imu_right_link</bodyName>
-        <updateRateHZ>100.0</updateRateHZ>
+        <updateRateHZ>${plugin_update_rate}</updateRateHZ>
         <gaussianNoise>0.0</gaussianNoise>
         <xyzOffset>0 0 0</xyzOffset>
@@ -239,9 +243,8 @@
   <gazebo>
     <plugin name="differential_drive_controller" filename="libgazebo_ros_diff_drive.so">
-      <legacyMode>true</legacyMode>
+      <legacyMode>false</legacyMode>
       <rosDebugLevel>Debug</rosDebugLevel>
-      <publishWheelTF>false</publishWheelTF>
       <robotNamespace>/</robotNamespace>
-      <publishTf>false</publishTf>
+      <publishTf>true</publishTf>
       <publishWheelJointState>false</publishWheelJointState>
       <alwaysOn>true</alwaysOn>
@@ -251,11 +254,11 @@
       <wheelSeparation>${2*base_radius}</wheelSeparation>
       <wheelDiameter>${2*wheel_radius}</wheelDiameter>
-      <broadcastTF>1</broadcastTF>
       <wheelTorque>30</wheelTorque>
       <wheelAcceleration>1.8</wheelAcceleration>
       <commandTopic>imcoders_keyboard_teleop/cmd_vel</commandTopic>
-      <odometryFrame>odom</odometryFrame>
-      <odometryTopic>odom</odometryTopic>
+      <odometryFrame>imcoders_odom</odometryFrame>
+      <odometryTopic>gazebo_odom</odometryTopic>
       <robotBaseFrame>base_footprint</robotBaseFrame>
+      <publishWheelTF>true</publishWheelTF>
     </plugin>
   </gazebo>
